Commit message: corrected typos in names

File: CPR_planar/cpr_planar_physics/launch/RERRFR/distal_plate.sdf.xacro (robot description, xacro)
@@ -16,5 +16,5 @@
     <xacro:arg name="x2" default="0.15"/>
     <xacro:arg name="y2" default="0"/>
-    <!--    Define the position of the joint for the second limb    -->
+    <!--    Define the position of the joint for the third limb    -->
     <xacro:arg name="x3" default="0"/>
     <xacro:arg name="y3" default="0"/>
@@ -126,5 +126,5 @@
             </geometry>
         </collision>
-        <visual name="limb1_attach_point_visual">
+        <!--<visual name="limb1_attach_point_visual">
             <geometry>
                 <box>
@@ -138,5 +138,5 @@
                </script>
             </material>
-        </visual>
+        </visual>-->
         <inertial>
             <mass>${mass/100}</mass>
@@ -212,5 +212,5 @@
             </geometry>
         </collision>
-        <visual name="limb2_attach_point_visual">
+<!--        <visual name="limb2_attach_point_visual">
             <geometry>
                 <box>
@@ -224,5 +224,5 @@
                </script>
             </material>
-        </visual>
+        </visual>-->
         <inertial>
             <mass>${mass/100}</mass>
@@ -293,5 +293,5 @@
         </geometry>
     </collision>
-    <visual name="limb3_attach_point_visual">
+    <!--<visual name="limb3_attach_point_visual">
         <geometry>
             <box>
@@ -305,5 +305,5 @@
            </script>
         </material>
-    </visual>
+    </visual>-->
     <inertial>
         <mass>${mass/100}</mass>
